File: xc9536xlBreakout-kicad/XC9536XL.sch (KiCad schematic (older format))
At the start: 29 parts, among them J1 19-36, J2 Conn_01x01, J3 JTAG, J4 Conn_01x03, J5 Conn_01x06, SW1 SW_DIP_x04, U1 XC9536XL-VQ44, U2 MIC5504-3.3YM5

Commit message: Add files via upload
6.9.21 After Design Review
Notes
Check forward current/ voltage on LEDs
reassign led resistor values to be lower
throw in some other sized caps for vcc
make caps as close as possible to each power pin
osc should be on power side as close as possible to to uC
Connections:
- net P1-6: now also J5.4 (Pin_4); no longer J5.3 (Pin_3)
- net P1-7: now also J5.3 (Pin_3); no longer J5.4 (Pin_4)
- net P2-3: now also U1.37 (P2-4); no longer U1.36 (GTS1/P2-3)
- net P2-4: now also U1.36 (GTS1/P2-3); no longer U1.37 (P2-4)
Changed lines of the file:
@@
-	1    0    0    -1
-$EndComp
-$Comp
-L xc9536xl-vq44:XC9536XL-VQ44 U1
-U 1 1 5DB36FFD
-P 6500 3500
-F 0 "U1" H 5900 4600 50  0000 C CNN
-F 1 "XC9536XL-VQ44" H 6500 2600 50  0000 C CNN
-F 2 "Package_QFP:TQFP-44_10x10mm_P0.8mm" H 6500 3500 50  0001 C CNN
-F 3 "" H 6500 3500 50  0001 C CNN
-	1    6500 3500
 	1    0    0    -1
 $EndComp
@@
 	5100 3000 5700 3000
 Wire Wire Line
-	5100 3100 5700 3100
-Wire Wire Line
-	5100 3200 5700 3200
-Wire Wire Line
 	5100 3300 5700 3300
 Wire Wire Line
@@
 Wire Wire Line
 	7300 2700 7900 2700
-Wire Wire Line
-	7300 2800 7900 2800
-Wire Wire Line
-	7300 2900 7900 2900
 Wire Wire Line
 	7300 3000 7900 3000
@@
 	7850 2500 7900 2500
 Wire Wire Line
-	6400 5050 6400 5200
-Wire Wire Line
 	6400 5200 6500 5200
-Wire Wire Line
-	6600 5200 6600 5050
-Wire Wire Line
-	6500 5050 6500 5200
 Connection ~ 6500 5200
 Wire Wire Line
@@
 Text Label 5300 3000 0    50   ~ 0
 P1-5
-Text Label 5300 3100 0    50   ~ 0
+Text Label 5100 3100 0    50   ~ 0
+P1-7
+Text Label 5100 3200 0    50   ~ 0
 P1-6
-Text Label 5300 3200 0    50   ~ 0
-P1-7
 Text Label 5300 3300 0    50   ~ 0
 P1-8
@@
 Text Label 7500 2700 0    50   ~ 0
 P2-2
-Text Label 7500 2800 0    50   ~ 0
+Text Label 7300 2900 0    50   ~ 0
 P2-3
-Text Label 7500 2900 0    50   ~ 0
+Text Label 7300 2800 0    50   ~ 0
 P2-4
 Text Label 7500 3000 0    50   ~ 0
@@
 Wire Wire Line
 	2600 5650 2400 5650
+Wire Wire Line
+	6600 5200 6600 5050
+Wire Wire Line
+	6500 5050 6500 5200
+Wire Wire Line
+	6400 5050 6400 5200
+$Comp
+L xc9536xl-vq44:XC9536XL-VQ44 U1
+U 1 1 5DB36FFD
+P 6500 3500
+F 0 "U1" H 5900 4600 50  0000 C CNN
+F 1 "XC9536XL-VQ44" H 6500 2600 50  0000 C CNN
+F 2 "Package_QFP:TQFP-44_10x10mm_P0.8mm" H 6500 3500 50  0001 C CNN
+F 3 "" H 6500 3500 50  0001 C CNN
+	1    6500 3500
+	1    0    0    -1
+$EndComp
+Wire Wire Line
+	5650 3100 5700 3100
+Text Label 5700 3200 2    50   ~ 0
+P1-7
+Text Label 5650 3100 2    50   ~ 0
+P1-6
+Text Label 7900 2900 2    50   ~ 0
+P2-4
+Text Label 7900 2800 2    50   ~ 0
+P2-3
 $EndSCHEMATC
